Commit message: trained model with horizontal arm

File: egomimic/resources/jaka_s12_pinza_nera_real_joints.urdf (robot description, URDF)
Before this commit: robot jaka_s12, 9 links, 8 joints
Joints:
- joint joint_5: origin xyz=0 -0.115 0 rpy=1.5708 0 0 -> xyz=0 -0.115 -0.1 rpy=1.5708 0 0

Commit message: various fix

File: egomimic/resources/jaka_s12_pinza_nera_real_joints.urdf (robot description, URDF)
Before this commit: robot jaka_s12, 9 links, 8 joints
Joints:
- joint joint_4: origin xyz=0.5715 0 0.1315 rpy=0 0 0 -> xyz=0.5715 0 0.0685 rpy=0 0 0
- joint joint_5: origin xyz=0 -0.115 -0.1 rpy=1.5708 0 0 -> xyz=0 -0.115 0 rpy=1.5708 0 0
